File: PCB Files/Kao Light Test Surface Mount.sch (EAGLE design)
At the start: 14 parts, among them T1 2N2222, Y1 16MHz

Commit message: feat: Adds status LEDs and Logo
Adds LEDs to indicate power from either the programming arduino's 5V
output or from the 5V regulator on the PCB. The LEDs should be different
colors and are labeled on the board. The logo is of the iSens logo
Parts:
- removed T1: 2N2222, adafruit:2N2222
- added FOOT_PEDAL: TP2P2-38-17, testpad:TP2P2-38-17
- added H1, H2, H3: MOUNT-PAD-ROUND2.8, holes:MOUNT-PAD-ROUND2.8
- added LASER_SWITCH: 2N3904, adafruit:2N2222
- added POWER, UPLOAD: (no value), adafruit:LEDCHIPLED_0805
- added R17, R18: 220, SparkFun-Resistors:200OHM-0603-1/10W-1%
- R16: value 200 -> 220
Connections:
- new net N$5: POWER.C, R17.2
- new net N$7: R18.2, UPLOAD.C
- net 5VOUT: now also FOOT_PEDALA.TP, POWER.A
- net GND: now also FOOT_PEDALB.TP, H1.MOUNT, H2.MOUNT, H3.MOUNT, LASER_SWITCH.E, POWER.3, R17.1, R18.1; no longer T1.E
- net N$2: now also LASER_SWITCH.B; no longer T1.B
- net N$3: now also LASER_SWITCH.C; no longer T1.C
- net RESET: now also POWER.1, R17.2
- net VIN: now also POWER.2, R17.1, UPLOAD.A
Other:
- moved on the sheet: LASER, R15, R16
